File: pcb/atari-junior-av-mod.kicad_pcb (KiCad board)
At the start: 2 copper layers, 94 x 89.5 mm, 337 parts

Commit message: Export 043c1d1 gerbers
Other:
- board text added: "043c1d1"
- board text removed: "f8384e4"
Changed lines of the file:
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@@
     (effects (font (size 0.8 0.8) (thickness 0.12)))
   )
-  (gr_text "f8384e4" (at 188.375 135.7355) (layer "F.SilkS")
+  (gr_text "043c1d1" (at 188.375 135.7355) (layer "F.SilkS")
     (effects (font (size 0.8 0.8) (thickness 0.12)))
   )
